File: sinktheship.brd (EAGLE design)
At the start: 99.4 x 81.9 mm, 16 parts, among them U1 TXB0108PWR, U2 TXB0108PWR

Commit message: rework done
Parts:
- moved S4 48.9 mm to (80.6, 19.1), turned to 0 degrees
- moved JP2 46.7 mm to (17.8, 21.6), flipped to the bottom
- moved S3 43.0 mm to (71.8, 27.9), turned to 0 degrees
- moved S1 34.6 mm to (89.5, 27.9), turned to 0 degrees
- moved C2 30.0 mm to (41.3, 45.7)
- moved C1 29.9 mm to (34.9, 45.7)
- moved S5 28.4 mm to (84.5, 81.3), turned to 0 degrees
- moved S2 27.1 mm to (80.6, 35.6), turned to 0 degrees
- moved U2 17.3 mm to (53.3, 45.1)
- moved U1 16.9 mm to (52.7, 62.9)
- moved S6 15.1 mm to (74.3, 72.4), turned to 0 degrees
- moved C4 13.3 mm to (52.1, 55.9), flipped to the bottom, turned to 270 degrees
- moved JP1 11.9 mm to (25.4, 57.8)
- moved R2 5.85 mm to (31.1, 45.7), turned to 270 degrees
- moved C3 5.75 mm to (39.4, 55.2), turned to 270 degrees
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Routing:
- net N$3: track 67.0 -> 195.3 mm, vias 1 -> 2
- net N$32: track 43.5 -> 148.0 mm, vias 0 -> 2
- net N$31: track 61.9 -> 151.2 mm, vias 0 -> 2
- net N$30: track 69.5 -> 153.9 mm, vias 0 -> 2
- net VCCA: track 80.5 -> 159.2 mm, vias 5 -> 7
- net N$28: track 89.0 -> 166.1 mm, vias 0 -> 2
- net N$29: track 79.2 -> 153.3 mm
- net VCCB: track 64.3 -> 131.8 mm, vias 5 -> 3
- net N$35: track 56.8 -> 111.3 mm
- net N$21: track 342.8 -> 386.1 mm
- net N$26: track 31.7 -> 71.8 mm, vias 0 -> 2
- net N$9: track 134.3 -> 95.4 mm
- net N$27: track 34.8 -> 72.1 mm, vias 0 -> 2
- net N$2: track 43.1 -> 72.7 mm
- net N$4: track 41.2 -> 64.6 mm
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